File: kicad/Untitled.kicad_sch (KiCad schematic)
At the start: 11 parts, among them J1 output, J3 output, J4 output, J5 Ch1 Ground, J6 Ch2 Ground

Commit message: sim_measured add
Parts:
- R1: value 2.2K R -> 10K R
Changed lines of the file:
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@@
 			)
 		)
-		(property "Value" "2.2K R"
+		(property "Value" "10K R"
 			(at 74.93 101.6 90)
 			(show_name no)
